File: Main/PCB/PCBOFBEATPAD/PCBOFBEATPAD.kicad_sch (KiCad schematic)
At the start: 31 parts, among them J2 7_pin_conector, SW1 SW_Push, U4 ESP32-C3_SUPERMINI_TH

Commit message: Major Update (V2 RELEASE)
Parts:
- removed A1, A2, A3, A4, A5, A6, A7, A8, A9: ~, ESP32-C3_SUPERMINI_TH:2x2 connectorss, symbol CONNECTORS:2x2_conector
- removed J2: 7_pin_conector, ESP32-C3_SUPERMINI_TH:1.3 tft display, symbol Ra-02:7_pin_conector
- removed R9: R_Small, Resistor_THT:R_Axial_DIN0204_L3.6mm_D1.6mm_P5.08mm_Horizontal, symbol Device:R_Small
- removed SW1: SW_Push, Button_Switch_THT:SW_PUSH_6mm, symbol Switch:SW_Push
- removed U4: ESP32-C3_SUPERMINI_TH, ESP32-C3_SUPERMINI_TH:MODULE_ESP32-C3_SUPERMINI_TH, symbol ESP32-C3_SUPERMINI_TH:ESP32-C3_SUPERMINI_TH
- added C1, C2, C4, C9: 10uF, Capacitor_SMD:C_0805_2012Metric_Pad1.18x1.45mm_HandSolder, symbol Device:C
- added C10: 1uF, Capacitor_SMD:C_0805_2012Metric_Pad1.18x1.45mm_HandSolder, symbol Device:C
- added C3, C5, C6, C7, C8: 0u1F, Capacitor_SMD:C_0805_2012Metric_Pad1.18x1.45mm_HandSolder, symbol Device:C
- added D10, D12, D13: LESD5D5.0CT1G, LESD5D5.0CT1G:TVS_LESD5D5.0CT1G, symbol LESD5D5.0CT1G:LESD5D5.0CT1G
- added D11: 1N5819HW-7-F, 1N5819HW-7-F:SOD3715X145N, symbol 1N5819HW-7-F:1N5819HW-7-F
- added D15: LTST-C190KGKT, LTST-C190KGKT:LEDC1608X35N, symbol LTST-C190KGKT:LTST-C190KGKT
- added J1: TYPE-C-31-M-12, TYPE-C-31-M-12:HRO_TYPE-C-31-M-12, symbol TYPE-C-31-M-12:TYPE-C-31-M-12
- added J3: Conn_01x03, Connector_PinSocket_2.00mm:PinSocket_1x03_P2.00mm_Vertical, symbol Connector_Generic:Conn_01x03
- added JP1: ~, Adafruit:1X11_ROUND_76, symbol Library:HEADER-1X1176MIL
- added R10, R13, R14: 10k, Resistor_SMD:R_0603_1608Metric_Pad0.98x0.95mm_HandSolder, symbol Device:R_Small
- added R11, R9: 5k1, Resistor_SMD:R_0805_2012Metric_Pad1.20x1.40mm_HandSolder, symbol Device:R
- added R12: 75, Resistor_SMD:R_0805_2012Metric_Pad1.20x1.40mm_HandSolder, symbol Device:R_Small
- added R15: 10k, Resistor_SMD:R_0603_1608Metric_Pad0.98x0.95mm_HandSolder, symbol Device:R
- added SW1, SW2, SW3: PTS810_SJM_250_SMTR_LFS, BUTTONS:SW_PTS810_SJM_250_SMTR_LFS, symbol PTS810_SJM_250_SMTR_LFS:PTS810_SJM_250_SMTR_LFS
- added U1, U10, U11, U3, U5, U6, U7, U8, U9: ~, randomahhconnector:2 pin connector, symbol Randomahhpinconeectorrr:2_pin_solderable_
- added U12: ESP32-S3-WROOM-1-N16R2, ESP32-S3-WROOM-1-N16R2:XCVR_ESP32-S3-WROOM-1-N16R2, symbol ESP32-S3-WROOM-1-N16R2:ESP32-S3-WROOM-1-N16R2
- added U13: AMS1117-3.3, AMS1117-3.3:SOT229P700X180-4N, symbol AMS1117-3.3:AMS1117-3.3
- R1, R2, R3, R4, R5, R6, R7, R8: value R_Small -> 10k; footprint Resistor_THT:R_Axial_DIN0204_L3.6mm_D1.6mm_P5.08mm_Horizontal -> Resistor_SMD:R_0603_1608Metric_Pad0.98x0.95mm_HandSolder
Connections:
- net 3.3v: now also U2.2 (VCC), C3.1, C4.1, C8.1, C9.1, R12.1, R13.1, R14.1, R15.1, U1.1 (Pin1), U10.1 (Pin1), U11.1 (Pin1), U12.2 (3V3), U13.2 (VOUT), U3.1 (Pin1), U5.1 (Pin1), U6.1 (Pin1), U7.1 (Pin1), U8.1 (Pin1), U9.1 (Pin1)
- net GND: now also R1.2, R2.2, R3.2, R4.2, R5.2, R6.2, R7.2, R8.2, C1.2, C10.2, C2.2, C3.2, C4.2, C5.2, C8.2, C9.2, D10.1, D12.1, D13.1, D15.C, J1.A1_B12 (GND), J1.B1_A12 (GND), J1.S1 (SHIELD), J1.S2 (SHIELD), J1.S3 (SHIELD), J1.S4 (SHIELD), J3.1 (Pin_1), JP1.3, R10.2, R11.2, R9.2, SW1.3, SW1.4, U12.1 (GND), U12.40 (GND), U12.41_1 (GND), U12.41_2 (GND), U12.41_3 (GND), U12.41_4 (GND), U12.41_5 (GND), U12.41_6 (GND), U12.41_7 (GND), U12.41_8 (GND), U12.41_9 (GND), U13.1 (GND/ADJ)
- net GPIO0: now also C7.1, R14.2, SW2.3, SW2.4, U12.27 (IO0)
- net GPIO3: now also U12.15 (IO3)
- net GPIO4: now also U12.4 (IO4)
- net GPIO5: now also U12.5 (IO5)
- net GPIO6: now also U12.6 (IO6)
- net GPIO7: now also U12.7 (IO7)
- net SK MINI LED: now also U12.18 (IO10)
- net Y0: now also R10.1, U1.2 (Pin2); no longer R1.1
- net Y1: now also R1.1, U3.2 (Pin2); no longer R4.1
- net Y2: now also R2.1, U5.2 (Pin2); no longer R7.1
- net Y3: now also R3.1, U6.2 (Pin2); no longer R2.1
- net Y4: now also R4.1, U7.2 (Pin2); no longer R5.1
- net Y5: now also R5.1, U8.2 (Pin2); no longer R8.1
- net Y6: now also R6.1, U9.2 (Pin2); no longer R3.1
- net Y7: now also R7.1, U10.2 (Pin2); no longer R6.1
- net Y8: now also R8.1, U11.2 (Pin2)
- net VCC renamed VCC_5V
- net VCC_5V: now also C1.1, C2.1, C5.1, D11.C, J3.3 (Pin_3), JP1.1, U13.3 (VIN); no longer U2.2 (VCC)
- new net: D15.A, R12.2
- new net: J1.A5 (CC1), R9.1
- new net: C6.2, SW3.1, SW3.2
- new net: J1.B5 (CC2), R11.1
- new net: C7.2, SW2.1, SW2.2
- new net 3.3V: J3.2 (Pin_2)
- new net CHIP_PU: C10.1, C6.1, R13.2, R15.2, SW3.3, SW3.4, U12.3 (EN)
- new net CS_DISPLAY: JP1.7, U12.38 (IO2)
- new net D+: D13.2, J1.A6 (DP1), J1.B6 (DP2), U12.14 (IO20)
- new net D-: D12.2, J1.A7 (DN1), J1.B7 (DN2), U12.13 (IO19)
- new net DC_DISPLAY: JP1.9, U12.39 (IO1)
- new net GPIO 46 AND 0 ~ STRAPPING PIN: U12.16 (IO46)
- new net MOSI_DISPLAY: JP1.6, U12.8 (IO15)
- new net RST: JP1.8, U12.12 (IO8)
- new net SCK_DISPLAY: JP1.4, U12.17 (IO9)
- new net SW_PUSH: SW1.1, SW1.2, U12.19 (IO11)
- new net VBUS: D10.2, D11.A, J1.A4_B9 (VBUS), J1.B4_A9 (VBUS)
- no-connect marks 26 -> 11
Other:
- moved on the sheet: D1, D2, D3, D4, D5, D6, D7, D8, D9, U2
